Commit message: - Initial attempt to rotate the robot to face a detected wall/kerb. - Contains updated, and a bit messy, laser_ranges_class.py which is used to test code before being copied into wall_follower.py - Adds angles.py and tuple_slicing.py for testing merged laser scans, division of lasers by robot regions etc

File: Sweeper/sweep_bot/urdf/sensors/laser.xacro (robot description, xacro)
@@ -348,4 +348,5 @@
     </xacro:macro> -->
     <!-- ************************************************************** -->
+    <!-- Hokuyo Laser - LEFT -->
      <xacro:macro name="laser_left_alt">
         <gazebo reference="hokuyo_link_left">
@@ -359,6 +360,4 @@
                         <samples>2500</samples>
                         <resolution>1</resolution>
-                        <!-- <min_angle>-1.5</min_angle> -->
-                        <!-- <max_angle>1.5</max_angle> -->
                         <min_angle>-3.14</min_angle>
                         <max_angle>1.57</max_angle>
@@ -402,8 +401,5 @@
         </link>
         <joint name="laser_joint_left" type="fixed">
-            <!-- <origin xyz="0.5 0.25 -0.20" rpy="0.0 0.01 ${3.14/4}"/> -->
             <origin xyz="0.5 0.25 -0.2" rpy="0.0 0.01 ${3.14/2}"/>
-            <!-- <origin xyz="0.5 0.25 -0.20" rpy="0.0 0.0 4.71238898"/> -->
-            <!-- <origin xyz="2.5 0.25 -0.20" rpy="0.0 0.0 0"/> -->
             <parent link="chasis"/>
             <child link="hokuyo_link_left"/>
@@ -424,11 +420,9 @@
                         <min_angle>-3.14</min_angle>
                         <max_angle>1.57</max_angle>
-                        <!-- <min_angle>-1.57</min_angle> -->
-                        <!-- <max_angle>1.57</max_angle> -->
-                    </horizontal>
-                </scan>
-                <range>
-                    <min>0.10</min>
-                    <max>4.7</max>
+                    </horizontal>
+                </scan>
+                <range>
+                    <min>0.10</min>
+                    <max>5.0</max>
                     <resolution>0.05</resolution>
                 </range>
@@ -466,4 +460,5 @@
         <joint name="laser_joint_right" type="fixed">
             <origin xyz="-0.5 -0.25 -0.2" rpy="0 0.01 -${3.14/2}"/>
+            <!-- <origin xyz="-0.5 -0.25 0.3" rpy="0 0.01 -${3.14/2}"/> -->
             <parent link="chasis"/>
             <child link="hokuyo_link_right"/>
