Commit message: ...working...

File: Sweeper/sweep_bot/urdf/cleaner.xacro (robot description, xacro)
@@ -5,5 +5,5 @@
   <xacro:include filename="$(find sweep_bot)/urdf/sensors/MultiCamera.xacro"/>
   <xacro:include filename="$(find sweep_bot)/urdf/sensors/laser.xacro"/>
-  <xacro:include filename="$(find hector_sensors_description)/urdf/hokuyo_utm30lx.urdf.xacro"/>
+  <!-- <xacro:include filename="$(find hector_sensors_description)/urdf/hokuyo_utm30lx.urdf.xacro"/> -->
   <!-- body -->
   <xacro:property name="chasis_length" value="1.0"/>
@@ -51,7 +51,7 @@
   <xacro:wheel side="right" position="aft" flip='-1' alt='-1'/>
   <!-- HOKUYO as RPLIDAR -->
-  <xacro:hokuyo_utm30lx name="hokuyo_laser" parent="chasis" ros_topic="hokuyo_scan" update_rate="40" ray_count="1040" min_angle="130" max_angle="-130">
+  <!-- <xacro:hokuyo_utm30lx name="hokuyo_laser" parent="chasis" ros_topic="hokuyo_scan" update_rate="40" ray_count="1040" min_angle="130" max_angle="-130">
     <origin xyz="0 0 0.3" rpy="0 0 0" />
-  </xacro:hokuyo_utm30lx>
+  </xacro:hokuyo_utm30lx> -->
   <!-- MULTI-CAMERA -->
   <xacro:sweeper_cams/>
@@ -60,5 +60,5 @@
   <!-- <xacro:laser_top/> -->
   <!-- <xacro:laser_front/> -->
-  <xacro:laser_left/>
+  <!-- <xacro:laser_left/> -->
   <!-- <xacro:laser_right/> -->
   <!-- <xacro:laser_rear/> -->

File: Sweeper/sweep_bot/urdf/sensors/laser.xacro (robot description, xacro)
@@ -44,5 +44,5 @@
                 <origin xyz="0 0 0" rpy="0 0 0"/>
                 <geometry>
-                    <mesh filename="package://rrbot_description/meshes/hokuyo.dae"/>
+                    <!-- <mesh filename="package://rrbot_description/meshes/hokuyo.dae"/> -->
                 </geometry>
             </visual>
@@ -106,5 +106,5 @@
                 <origin xyz="0 0 0" rpy="0 0 0"/>
                 <geometry>
-                    <mesh filename="package://rrbot_description/meshes/hokuyo.dae"/>
+                    <!-- <mesh filename="package://rrbot_description/meshes/hokuyo.dae"/> -->
                 </geometry>
             </visual>
@@ -172,5 +172,8 @@
                 <origin xyz="0 0 0" rpy="0 0 0"/>
                 <geometry>
-                    <mesh filename="package://rrbot_description/meshes/hokuyo.dae"/>
+                    <!-- <mesh filename="package://rrbot_description/meshes/hokuyo.dae"/> -->
+                    <!-- <mesh filename="sweep_bot/meshes/hokuyo.dae"/> -->
+                    <mesh filename="package://sweep_bot/meshes/hokuyo.dae"/>
+                    <!-- <mesh filename="$(find sweep_bot)/meshes/hokuyo.dae"/> -->
                 </geometry>
             </visual>
@@ -234,5 +237,5 @@
                 <origin xyz="0 0 0" rpy="0 0 0"/>
                 <geometry>
-                    <mesh filename="package://rrbot_description/meshes/hokuyo.dae"/>
+                    <!-- <mesh filename="package://rrbot_description/meshes/hokuyo.dae"/> -->
                 </geometry>
             </visual>
@@ -295,5 +298,5 @@
                 <origin xyz="0 0 0" rpy="0 0 0"/>
                 <geometry>
-                    <mesh filename="package://rrbot_description/meshes/hokuyo.dae"/>
+                    <!-- <mesh filename="package://rrbot_description/meshes/hokuyo.dae"/> -->
                 </geometry>
             </visual>

Commit message: Updates xacro to include front laser Experiements with merging front with side lasers Adds workflow to the wall-follower script which helps the robot transition from stage to stage

File: Sweeper/sweep_bot/urdf/cleaner.xacro (robot description, xacro)
@@ -59,5 +59,5 @@
   <!-- LASERS -->
   <!-- <xacro:laser_top/> -->
-  <!-- <xacro:laser_front/> -->
+  <xacro:laser_front/>
   <xacro:laser_left/>
   <xacro:laser_right/>

File: Sweeper/sweep_bot/urdf/sensors/laser.xacro (robot description, xacro)
@@ -107,4 +107,5 @@
                 <geometry>
                     <!-- <mesh filename="package://rrbot_description/meshes/hokuyo.dae"/> -->
+                    <mesh filename="package://sweep_bot/meshes/hokuyo.dae"/>
                 </geometry>
             </visual>
@@ -117,7 +118,5 @@
         <joint name="laser_joint_front" type="fixed">
             <origin xyz="0.53 0 -0.20" rpy="0 0.0 0"/>
-            <!-- <origin xyz="0.53 0 -0.25" rpy="0 0.0 0"/> -->
-            <!-- <origin xyz="0.53 0 -0.22" rpy="0 0.0 0"/> -->
-            <!-- <origin xyz="0.53 0 0" rpy="0 0.0 0"/> -->
+            <!-- <origin xyz="0.53 0.05 -0.20" rpy="0 0.0 0"/> -->
             <parent link="chasis"/>
             <child link="hokuyo_link_front"/>
@@ -238,4 +237,5 @@
                 <geometry>
                     <!-- <mesh filename="package://rrbot_description/meshes/hokuyo.dae"/> -->
+                    <mesh filename="package://sweep_bot/meshes/hokuyo.dae"/>
                 </geometry>
             </visual>
@@ -299,4 +299,5 @@
                 <geometry>
                     <!-- <mesh filename="package://rrbot_description/meshes/hokuyo.dae"/> -->
+                    <mesh filename="package://sweep_bot/meshes/hokuyo.dae"/>
                 </geometry>
             </visual>

Commit message: - Reconfigured the position of the lasers on the robot to achieve "360 degress" coverage - merge_laser_scans.launch refactured to merge 2 laser topics, /scan_left and /scan_right - Amends experimental code in laser_ranges_class.py file to utilize the new configuration - Increases the sample rates by 50 times to eliminate the issue with intermittend laser ranging data - Removes experimental and ineffective parameters from merge_laser_scans launch file

File: Sweeper/sweep_bot/urdf/cleaner.xacro (robot description, xacro)
@@ -8,4 +8,5 @@
   <!-- body -->
   <xacro:property name="chasis_length" value="1.0"/>
+  <!-- <xacro:property name="chasis_width" value="0.45"/> -->
   <xacro:property name="chasis_width" value="0.45"/>
   <xacro:property name="chasis_heigth" value="0.5"/>
@@ -15,8 +16,29 @@
   <xacro:property name="izz" value="${(1/12 * chasis_mass) * ((chasis_heigth * chasis_heigth) + (chasis_width * chasis_width))}"/>
   <link name="chasis_footprint"/>
+  <!-- <link name="chasis_footprint">
+    <inertial>
+      <origin xyz="0.0 0.0 -0.5" rpy="0.0 1.57 0.0"/>
+      <mass value="${chasis_mass}"/>
+      <inertia ixx="${ixx}" ixy="0.0" ixz="0.0" iyy="${iyy}" iyz="0.0" izz="${izz}"/>
+    </inertial>
+    <visual name="">
+      <origin xyz="0.0 0.0 -0.5" rpy="0.0 0.0 0.0"/>
+      <geometry>
+        <box size="${chasis_length} ${chasis_width} ${chasis_heigth}"/>
+      </geometry>
+      <material name="">
+      </material>
+    </visual>
+    <collision>
+      <origin xyz="0.0 0.0 -0.5" rpy="0.0 0.0 0.0"/>
+      <geometry>
+        <box size="${chasis_length} ${chasis_width} ${chasis_heigth}"/>
+      </geometry>
+    </collision>
+  </link> -->
   <joint name="chasis_footprint_joint" type="fixed">
     <parent link="chasis_footprint"/>
     <child link="chasis"/>
-    <origin xyz="0.0 0.0 0.0" rpy="0.0 0.0 0.0"/>
+    <origin xyz="0.0 0.0 0.25" rpy="0.0 0.0 0.0"/>
   </joint>
   <link name="chasis">
@@ -37,7 +59,7 @@
     <collision>
       <origin xyz="0.0 0.0 0.0" rpy="0.0 0.0 0.0"/>
-      <geometry>
+      <!-- <geometry>
         <box size="${chasis_length} ${chasis_width} ${chasis_heigth}"/>
-      </geometry>
+      </geometry> -->
     </collision>
   </link>
@@ -59,7 +81,10 @@
   <!-- LASERS -->
   <!-- <xacro:laser_top/> -->
-  <xacro:laser_front/>
-  <xacro:laser_left/>
-  <xacro:laser_right/>
+  <!-- <xacro:laser_front/> -->
+  <!-- <xacro:laser_left/> -->
+  <!-- <xacro:laser_right/> -->
+  <xacro:laser_left_alt/>
+  <xacro:laser_right_alt/>
+  <!-- <xacro:laser_center/> -->
   <!-- <xacro:laser_rear/> -->
   <!-- SKIP STEERING -->

File: Sweeper/sweep_bot/urdf/sensors/laser.xacro (robot description, xacro)
@@ -3,5 +3,5 @@
     <!-- Hokuyo Laser - TOP -->
     <xacro:macro name="laser_top">
-        <!-- <gazebo reference="hokuyo_link_top">
+        <gazebo reference="hokuyo_link_top">
             <sensor type="ray" name="head_hokuyo_sensor">
             <pose>0 0 0 0 0 0</pose>
@@ -11,8 +11,8 @@
                 <scan>
                     <horizontal>
-                        <samples>720</samples>
-                        <resolution>1</resolution>
-                        <min_angle>-0.5</min_angle>
-                        <max_angle>0.5</max_angle>
+                        <samples>360</samples>
+                        <resolution>1</resolution>
+                        <min_angle>-3.14</min_angle>
+                        <max_angle>3.14</max_angle>
                     </horizontal>
                 </scan>
@@ -29,9 +29,9 @@
             </ray>
             <plugin name="gazebo_ros_head_hokuyo_controller" filename="libgazebo_ros_laser.so">
-                <topicName>/scan</topicName>
+                <topicName>/scans</topicName>
                 <frameName>hokuyo_link_top</frameName>
             </plugin>
             </sensor>
-        </gazebo> -->
+        </gazebo>
         <link name="hokuyo_link_top">
             <collision>
@@ -44,5 +44,4 @@
                 <origin xyz="0 0 0" rpy="0 0 0"/>
                 <geometry>
-                    <!-- <mesh filename="package://rrbot_description/meshes/hokuyo.dae"/> -->
                 </geometry>
             </visual>
@@ -65,5 +64,4 @@
             <pose>0 0 0 0 0 0</pose>
             <visualize>true</visualize>
-            <!-- <update_rate>20</update_rate> -->
             <update_rate>20</update_rate>
             <ray>
@@ -72,6 +70,4 @@
                         <samples>50</samples>
                         <resolution>1</resolution>
-                        <!-- <min_angle>-1.570796</min_angle> -->
-                        <!-- <max_angle>1.570796</max_angle> -->
                         <min_angle>-1.5</min_angle>
                         <max_angle>1.5</max_angle>
@@ -95,5 +91,4 @@
             </sensor>
         </gazebo>
-        <!--  -->
         <link name="hokuyo_link_front">
             <collision>
@@ -106,5 +101,4 @@
                 <origin xyz="0 0 0" rpy="0 0 0"/>
                 <geometry>
-                    <!-- <mesh filename="package://rrbot_description/meshes/hokuyo.dae"/> -->
                     <mesh filename="package://sweep_bot/meshes/hokuyo.dae"/>
                 </geometry>
@@ -118,9 +112,65 @@
         <joint name="laser_joint_front" type="fixed">
             <origin xyz="0.53 0 -0.20" rpy="0 0.0 0"/>
-            <!-- <origin xyz="0.53 0.05 -0.20" rpy="0 0.0 0"/> -->
             <parent link="chasis"/>
             <child link="hokuyo_link_front"/>
         </joint>
     </xacro:macro>
+<!-- Hokuyo Laser - CENTER -->
+    <!-- <xacro:macro name="laser_center">
+        <gazebo reference="hokuyo_link_center">
+            <sensor type="ray" name="head_hokuyo_sensor">
+            <pose>0 0 0 0 0 0</pose>
+            <visualize>true</visualize>
+            <update_rate>20</update_rate>
+            <ray>
+                <scan>
+                    <horizontal>
+                        <samples>360</samples>
+                        <resolution>1</resolution>
+                        <min_angle>-3.14</min_angle>
+                        <max_angle>3.14</max_angle>
+                    </horizontal>
+                </scan>
+                <range>
+                    <min>0.10</min>
+                    <max>10.0</max>
+                    <resolution>0.05</resolution>
+                </range>
+                <noise>
+                    <type>gaussian</type>
+                    <mean>0.0</mean>
+                    <stddev>0.01</stddev>
+                </noise>
+            </ray>
+            <plugin name="gazebo_ros_head_hokuyo_controller" filename="libgazebo_ros_laser.so">
+                <topicName>/scan_center</topicName>
+                <frameName>hokuyo_link_center</frameName>
+            </plugin>
+            </sensor>
+        </gazebo>
+        <link name="hokuyo_link_center">
+            <collision>
+                <origin xyz="0 0 0" rpy="0 0 0"/>
+                <geometry>
+                    <box size="0.1 0.1 0.1"/>
+                </geometry>
+            </collision>
+            <visual>
+                <origin xyz="0 0 0" rpy="0 0 0"/>
+                <geometry>
+                </geometry>
+            </visual>
+            <inertial>
+                <mass value="1e-5" />
+                <origin xyz="0 0 0" rpy="0 0 0"/>
+                <inertia ixx="1e-6" ixy="0" ixz="0" iyy="1e-6" iyz="0" izz="1e-6" />
+            </inertial>
+        </link>
+        <joint name="laser_joint_center" type="fixed">
+            <origin xyz="0.0 0 -0.28" rpy="0 0 0"/>
+            <parent link="chasis"/>
+            <child link="hokuyo_link_center"/>
+        </joint>
+    </xacro:macro> -->
     <!-- Hokuyo Laser - LEFT -->
     <xacro:macro name="laser_left">
@@ -135,10 +185,6 @@
                         <samples>50</samples>
                         <resolution>1</resolution>
-                        <!-- <min_angle>-1.570796</min_angle> -->
-                        <!-- <max_angle>1.570796</max_angle> -->
                         <min_angle>-1.5</min_angle>
                         <max_angle>1.5</max_angle>
-                        <!-- <min_angle>-0.2</min_angle> -->
-                        <!-- <max_angle>0.2</max_angle> -->
                     </horizontal>
                 </scan>
@@ -160,5 +206,4 @@
             </sensor>
         </gazebo>
-        <!--  -->
         <link name="hokuyo_link_left">
             <collision>
@@ -171,8 +216,5 @@
                 <origin xyz="0 0 0" rpy="0 0 0"/>
                 <geometry>
-                    <!-- <mesh filename="package://rrbot_description/meshes/hokuyo.dae"/> -->
-                    <!-- <mesh filename="sweep_bot/meshes/hokuyo.dae"/> -->
-                    <mesh filename="package://sweep_bot/meshes/hokuyo.dae"/>
-                    <!-- <mesh filename="$(find sweep_bot)/meshes/hokuyo.dae"/> -->
+                    <mesh filename="package://sweep_bot/meshes/hokuyo.dae"/>
                 </geometry>
             </visual>
@@ -184,5 +226,4 @@
         </link>
         <joint name="laser_joint_left" type="fixed">
-            <!-- <origin xyz="0.0 0.25 0.29" rpy="-0.5 0 0"/> -->
             <origin xyz="0.0 0.25 -0.20" rpy="0 0.01 ${3.14/2}"/>
             <parent link="chasis"/>
@@ -202,6 +243,4 @@
                         <samples>50</samples>
                         <resolution>1</resolution>
-                        <!-- <min_angle>-1.570796</min_angle> -->
-                        <!-- <max_angle>1.570796</max_angle> -->
                         <min_angle>-1.5</min_angle>
                         <max_angle>1.5</max_angle>
@@ -225,5 +264,4 @@
             </sensor>
         </gazebo>
-        <!--  -->
         <link name="hokuyo_link_right">
             <collision>
@@ -236,5 +274,4 @@
                 <origin xyz="0 0 0" rpy="0 0 0"/>
                 <geometry>
-                    <!-- <mesh filename="package://rrbot_description/meshes/hokuyo.dae"/> -->
                     <mesh filename="package://sweep_bot/meshes/hokuyo.dae"/>
                 </geometry>
@@ -253,5 +290,5 @@
     </xacro:macro>
     <!-- Hokuyo Laser - REAR -->
-    <xacro:macro name="laser_rear">
+    <!-- <xacro:macro name="laser_rear">
         <gazebo reference="hokuyo_link_rear">
             <sensor type="ray" name="head_hokuyo_sensor_rear">
@@ -264,6 +301,4 @@
                         <samples>720</samples>
                         <resolution>1</resolution>
-                        <!-- <min_angle>-1.570796</min_angle> -->
-                        <!-- <max_angle>1.570796</max_angle> -->
                         <min_angle>-1.5</min_angle>
                         <max_angle>1.5</max_angle>
@@ -287,5 +322,4 @@
             </sensor>
         </gazebo>
-        <!--  -->
         <link name="hokuyo_link_rear">
             <collision>
@@ -298,5 +332,4 @@
                 <origin xyz="0 0 0" rpy="0 0 0"/>
                 <geometry>
-                    <!-- <mesh filename="package://rrbot_description/meshes/hokuyo.dae"/> -->
                     <mesh filename="package://sweep_bot/meshes/hokuyo.dae"/>
                 </geometry>
@@ -313,4 +346,127 @@
             <child link="hokuyo_link_rear"/>
         </joint>
+    </xacro:macro> -->
+    <!-- ************************************************************** -->
+     <xacro:macro name="laser_left_alt">
+        <gazebo reference="hokuyo_link_left">
+            <sensor type="ray" name="head_hokuyo_sensor_left">
+            <pose>0 0 0 0 0 0</pose>
+            <visualize>true</visualize>
+            <update_rate>20</update_rate>
+            <ray>
+                <scan>
+                    <horizontal>
+                        <samples>2500</samples>
+                        <resolution>1</resolution>
+                        <!-- <min_angle>-1.5</min_angle> -->
+                        <!-- <max_angle>1.5</max_angle> -->
+                        <min_angle>-3.14</min_angle>
+                        <max_angle>1.57</max_angle>
+                    </horizontal>
+                </scan>
+                <range>
+                    <min>0.10</min>
+                    <max>5.0</max>
+                    <resolution>0.05</resolution>
+                </range>
+                <noise>
+                    <type>gaussian</type>
+                    <mean>0.0</mean>
+                    <stddev>0.01</stddev>
+                </noise>
+            </ray>
+            <plugin name="gazebo_ros_head_hokuyo_controller" filename="libgazebo_ros_laser.so">
+                <topicName>/scan_left</topicName>
+                <frameName>hokuyo_link_left</frameName>
+            </plugin>
+            </sensor>
+        </gazebo>
+        <link name="hokuyo_link_left">
+            <collision>
+                <origin xyz="0 0 0" rpy="0 0 0"/>
+                <geometry>
+                    <box size="0.1 0.1 0.1"/>
+                </geometry>
+            </collision>
+            <visual>
+                <origin xyz="0 0 0" rpy="0 0 0"/>
+                <geometry>
+                    <mesh filename="package://sweep_bot/meshes/hokuyo.dae"/>
+                </geometry>
+            </visual>
+            <inertial>
+                <mass value="1e-5" />
+                <origin xyz="0 0 0" rpy="0 0 0"/>
+                <inertia ixx="1e-6" ixy="0" ixz="0" iyy="1e-6" iyz="0" izz="1e-6" />
+            </inertial>
+        </link>
+        <joint name="laser_joint_left" type="fixed">
+            <!-- <origin xyz="0.5 0.25 -0.20" rpy="0.0 0.01 ${3.14/4}"/> -->
+            <origin xyz="0.5 0.25 -0.2" rpy="0.0 0.01 ${3.14/2}"/>
+            <!-- <origin xyz="0.5 0.25 -0.20" rpy="0.0 0.0 4.71238898"/> -->
+            <!-- <origin xyz="2.5 0.25 -0.20" rpy="0.0 0.0 0"/> -->
+            <parent link="chasis"/>
+            <child link="hokuyo_link_left"/>
+        </joint>
+    </xacro:macro>
+    <!-- Hokuyo Laser - RIGHT -->
+    <xacro:macro name="laser_right_alt">
+        <gazebo reference="hokuyo_link_right">
+            <sensor type="ray" name="head_hokuyo_sensor_right">
+            <pose>0 0 0 0 0 0</pose>
+            <visualize>true</visualize>
+            <update_rate>20</update_rate>
+            <ray>
+                <scan>
+                    <horizontal>
+                        <samples>2500</samples>
+                        <resolution>1</resolution>
+                        <min_angle>-3.14</min_angle>
+                        <max_angle>1.57</max_angle>
+                        <!-- <min_angle>-1.57</min_angle> -->
+                        <!-- <max_angle>1.57</max_angle> -->
+                    </horizontal>
+                </scan>
+                <range>
+                    <min>0.10</min>
+                    <max>4.7</max>
+                    <resolution>0.05</resolution>
+                </range>
+                <noise>
+                    <type>gaussian</type>
+                    <mean>0.0</mean>
+                    <stddev>0.01</stddev>
+                </noise>
+            </ray>
+            <plugin name="gazebo_ros_head_hokuyo_controller" filename="libgazebo_ros_laser.so">
+                <topicName>/scan_right</topicName>
+                <frameName>hokuyo_link_right</frameName>
+            </plugin>
+            </sensor>
+        </gazebo>
+        <link name="hokuyo_link_right">
+            <collision>
+                <origin xyz="0 0 0" rpy="0 0 0"/>
+                <geometry>
+                    <box size="0.1 0.1 0.1"/>
+                </geometry>
+            </collision>
+            <visual>
+                <origin xyz="0 0 0" rpy="0 0 0"/>
+                <geometry>
+                    <mesh filename="package://sweep_bot/meshes/hokuyo.dae"/>
+                </geometry>
+            </visual>
+            <inertial>
+                <mass value="1e-5" />
+                <origin xyz="0 0 0" rpy="0 0 0"/>
+                <inertia ixx="1e-6" ixy="0" ixz="0" iyy="1e-6" iyz="0" izz="1e-6" />
+            </inertial>
+        </link>
+        <joint name="laser_joint_right" type="fixed">
+            <origin xyz="-0.5 -0.25 -0.2" rpy="0 0.01 -${3.14/2}"/>
+            <parent link="chasis"/>
+            <child link="hokuyo_link_right"/>
+        </joint>
     </xacro:macro>
 </robot>
