Commit message: Creates settings.py for centralized definition of variables data and imports into core logic python scripts Began using some variables from settings.py Adds extra distance variables to angles.msg to indicate distance to right wall Updates laser_ranges_class test script with PID-functions experimenting with various situations especially the wall following in the pidLine() function Amends city world for quicker loading Reduces laser radius from 26.0 to 6.0 to better fit into the test city

File: Sweeper/sweep_bot/urdf/cleaner.xacro (robot description, xacro)
@@ -59,7 +59,7 @@
     <collision>
       <origin xyz="0.0 0.0 0.0" rpy="0.0 0.0 0.0"/>
-      <!-- <geometry>
+      <geometry>
         <box size="${chasis_length} ${chasis_width} ${chasis_heigth}"/>
-      </geometry> -->
+      </geometry>
     </collision>
   </link>
@@ -80,12 +80,6 @@
   <!-- <xacro:overwatch_cam/> -->
   <!-- LASERS -->
-  <!-- <xacro:laser_top/> -->
-  <!-- <xacro:laser_front/> -->
-  <!-- <xacro:laser_left/> -->
-  <!-- <xacro:laser_right/> -->
   <xacro:laser_left_alt/>
   <xacro:laser_right_alt/>
-  <!-- <xacro:laser_center/> -->
-  <!-- <xacro:laser_rear/> -->
   <!-- SKIP STEERING -->
   <gazebo>

File: Sweeper/sweep_bot/urdf/sensors/laser.xacro (robot description, xacro)
@@ -349,5 +349,5 @@
     <!-- ************************************************************** -->
     <!-- Hokuyo Laser - LEFT -->
-     <xacro:macro name="laser_left_alt">
+    <xacro:macro name="laser_left_alt">
         <gazebo reference="hokuyo_link_left">
             <sensor type="ray" name="head_hokuyo_sensor_left">
@@ -366,5 +366,5 @@
                 <range>
                     <min>0.10</min>
-                    <max>5.0</max>
+                    <max>2.5</max>
                     <resolution>0.05</resolution>
                 </range>
@@ -401,5 +401,7 @@
         </link>
         <joint name="laser_joint_left" type="fixed">
-            <origin xyz="0.5 0.25 -0.2" rpy="0.0 0.01 ${3.14/2}"/>
+            <!-- <origin xyz="0.5 0.25 -0.2" rpy="0.0 0.01 ${3.14/2}"/> -->
+            <!-- <origin xyz="0.53 0.25 0.2" rpy="0.0 0.01 ${3.14/2}"/> -->
+            <origin xyz="0.56 0.28 0.2" rpy="0.0 0.0 ${3.14/2}"/>
             <parent link="chasis"/>
             <child link="hokuyo_link_left"/>
@@ -424,5 +426,5 @@
                 <range>
                     <min>0.10</min>
-                    <max>5.0</max>
+                    <max>2.5</max>
                     <resolution>0.05</resolution>
                 </range>
@@ -459,6 +461,7 @@
         </link>
         <joint name="laser_joint_right" type="fixed">
-            <origin xyz="-0.5 -0.25 -0.2" rpy="0 0.01 -${3.14/2}"/>
-            <!-- <origin xyz="-0.5 -0.25 0.3" rpy="0 0.01 -${3.14/2}"/> -->
+            <!-- <origin xyz="-0.5 -0.25 -0.2" rpy="0 0.01 -${3.14/2}"/> -->
+            <!-- <origin xyz="-0.53 -0.25 0.2" rpy="0.0 0.01 -${3.14/2}"/> -->
+            <origin xyz="-0.56 -0.28 0.2" rpy="0.0 0.0 -${3.14/2}"/>
             <parent link="chasis"/>
             <child link="hokuyo_link_right"/>

Commit message: General clean up of wall-follower.py Resets street sidewalk height back to original value BUT increases it slightly again as robot failed to detect bow mid-distance and stop robot when finding-right-wall Clean up of cleaner.xacro, drive.launch and other resources

File: Sweeper/sweep_bot/urdf/cleaner.xacro (robot description, xacro)
@@ -5,8 +5,6 @@
   <xacro:include filename="$(find sweep_bot)/urdf/sensors/MultiCamera.xacro"/>
   <xacro:include filename="$(find sweep_bot)/urdf/sensors/laser.xacro"/>
-  <!-- <xacro:include filename="$(find hector_sensors_description)/urdf/hokuyo_utm30lx.urdf.xacro"/> -->
   <!-- body -->
   <xacro:property name="chasis_length" value="1.0"/>
-  <!-- <xacro:property name="chasis_width" value="0.45"/> -->
   <xacro:property name="chasis_width" value="0.45"/>
   <xacro:property name="chasis_heigth" value="0.5"/>
@@ -16,25 +14,4 @@
   <xacro:property name="izz" value="${(1/12 * chasis_mass) * ((chasis_heigth * chasis_heigth) + (chasis_width * chasis_width))}"/>
   <link name="chasis_footprint"/>
-  <!-- <link name="chasis_footprint">
-    <inertial>
-      <origin xyz="0.0 0.0 -0.5" rpy="0.0 1.57 0.0"/>
-      <mass value="${chasis_mass}"/>
-      <inertia ixx="${ixx}" ixy="0.0" ixz="0.0" iyy="${iyy}" iyz="0.0" izz="${izz}"/>
-    </inertial>
-    <visual name="">
-      <origin xyz="0.0 0.0 -0.5" rpy="0.0 0.0 0.0"/>
-      <geometry>
-        <box size="${chasis_length} ${chasis_width} ${chasis_heigth}"/>
-      </geometry>
-      <material name="">
-      </material>
-    </visual>
-    <collision>
-      <origin xyz="0.0 0.0 -0.5" rpy="0.0 0.0 0.0"/>
-      <geometry>
-        <box size="${chasis_length} ${chasis_width} ${chasis_heigth}"/>
-      </geometry>
-    </collision>
-  </link> -->
   <joint name="chasis_footprint_joint" type="fixed">
     <parent link="chasis_footprint"/>
@@ -72,11 +49,6 @@
   <xacro:wheel side="left" position="aft" flip='1' alt='-1'/>
   <xacro:wheel side="right" position="aft" flip='-1' alt='-1'/>
-  <!-- HOKUYO as RPLIDAR -->
-  <!-- <xacro:hokuyo_utm30lx name="hokuyo_laser" parent="chasis" ros_topic="hokuyo_scan" update_rate="40" ray_count="1040" min_angle="130" max_angle="-130">
-    <origin xyz="0 0 0.3" rpy="0 0 0" />
-  </xacro:hokuyo_utm30lx> -->
   <!-- MULTI-CAMERA -->
   <xacro:sweeper_cams/>
-  <!-- <xacro:overwatch_cam/> -->
   <!-- LASERS -->
   <xacro:laser_left_alt/>
@@ -107,24 +79,4 @@
   <!--  -->
   <!-- IMU -->
-  <!-- <gazebo reference="imu_link">
-    <gravity>true</gravity>
-    <sensor name="imu_sensor" type="imu">
-      <always_on>true</always_on>
-      <update_rate>100</update_rate>
-      <visualize>true</visualize>
-      <topic>__default_topic__</topic>
-      <plugin filename="libgazebo_ros_imu_sensor.so" name="imu_plugin">
-        <topicName>imu</topicName>
-        <bodyName>imu_link</bodyName>
-        <updateRateHZ>10.0</updateRateHZ>
-        <gaussianNoise>0.0</gaussianNoise>
-        <xyzOffset>0 0 0</xyzOffset>
-        <rpyOffset>0 0 0</rpyOffset>
-        <frameName>imu_link</frameName>
-        <initialOrientationAsReference>false</initialOrientationAsReference>
-      </plugin>
-      <pose>0 0 0 0 0 0</pose>
-    </sensor>
-  </gazebo> -->
   <gazebo>
     <plugin name="imu_plugin" filename="libgazebo_ros_imu.so">

File: Sweeper/sweep_bot/urdf/sensors/laser.xacro (robot description, xacro)
@@ -1,351 +1,4 @@
 <?xml version="1.0"?>
 <robot xmlns:xacro="http://www.ros.org/wiki/xacro" name="robot_name">
-    <!-- Hokuyo Laser - TOP -->
-    <xacro:macro name="laser_top">
-        <gazebo reference="hokuyo_link_top">
-            <sensor type="ray" name="head_hokuyo_sensor">
-            <pose>0 0 0 0 0 0</pose>
-            <visualize>true</visualize>
-            <update_rate>20</update_rate>
-            <ray>
-                <scan>
-                    <horizontal>
-                        <samples>360</samples>
-                        <resolution>1</resolution>
-                        <min_angle>-3.14</min_angle>
-                        <max_angle>3.14</max_angle>
-                    </horizontal>
-                </scan>
-                <range>
-                    <min>0.10</min>
-                    <max>10.0</max>
-                    <resolution>0.05</resolution>
-                </range>
-                <noise>
-                    <type>gaussian</type>
-                    <mean>0.0</mean>
-                    <stddev>0.01</stddev>
-                </noise>
-            </ray>
-            <plugin name="gazebo_ros_head_hokuyo_controller" filename="libgazebo_ros_laser.so">
-                <topicName>/scans</topicName>
-                <frameName>hokuyo_link_top</frameName>
-            </plugin>
-            </sensor>
-        </gazebo>
-        <link name="hokuyo_link_top">
-            <collision>
-                <origin xyz="0 0 0" rpy="0 0 0"/>
-                <geometry>
-                    <box size="0.1 0.1 0.1"/>
-                </geometry>
-            </collision>
-            <visual>
-                <origin xyz="0 0 0" rpy="0 0 0"/>
-                <geometry>
-                </geometry>
-            </visual>
-            <inertial>
-                <mass value="1e-5" />
-                <origin xyz="0 0 0" rpy="0 0 0"/>
-                <inertia ixx="1e-6" ixy="0" ixz="0" iyy="1e-6" iyz="0" izz="1e-6" />
-            </inertial>
-        </link>
-        <joint name="laser_joint_top" type="fixed">
-            <origin xyz="0.0 0 0.29" rpy="0 0 0"/>
-            <parent link="chasis"/>
-            <child link="hokuyo_link_top"/>
-        </joint>
-    </xacro:macro>
-    <!-- Hokuyo Laser - FRONT -->
-    <xacro:macro name="laser_front">
-        <gazebo reference="hokuyo_link_front">
-            <sensor type="ray" name="head_hokuyo_sensor_front">
-            <pose>0 0 0 0 0 0</pose>
-            <visualize>true</visualize>
-            <update_rate>20</update_rate>
-            <ray>
-                <scan>
-                    <horizontal>
-                        <samples>50</samples>
-                        <resolution>1</resolution>
-                        <min_angle>-1.5</min_angle>
-                        <max_angle>1.5</max_angle>
-                    </horizontal>
-                </scan>
-                <range>
-                    <min>0.10</min>
-                    <max>10</max>
-                    <resolution>0.05</resolution>
-                </range>
-                <noise>
-                    <type>gaussian</type>
-                    <mean>0.0</mean>
-                    <stddev>0.01</stddev>
-                </noise>
-            </ray>
-            <plugin name="gazebo_ros_head_hokuyo_controller" filename="libgazebo_ros_laser.so">
-                <topicName>/scan_front</topicName>
-                <frameName>hokuyo_link_front</frameName>
-            </plugin>
-            </sensor>
-        </gazebo>
-        <link name="hokuyo_link_front">
-            <collision>
-                <origin xyz="0 0 0" rpy="0 0 0"/>
-                <geometry>
-                    <box size="0.1 0.1 0.1"/>
-                </geometry>
-            </collision>
-            <visual>
-                <origin xyz="0 0 0" rpy="0 0 0"/>
-                <geometry>
-                    <mesh filename="package://sweep_bot/meshes/hokuyo.dae"/>
-                </geometry>
-            </visual>
-            <inertial>
-                <mass value="1e-5" />
-                <origin xyz="0 0 0" rpy="0 0 0"/>
-                <inertia ixx="1e-6" ixy="0" ixz="0" iyy="1e-6" iyz="0" izz="1e-6" />
-            </inertial>
-        </link>
-        <joint name="laser_joint_front" type="fixed">
-            <origin xyz="0.53 0 -0.20" rpy="0 0.0 0"/>
-            <parent link="chasis"/>
-            <child link="hokuyo_link_front"/>
-        </joint>
-    </xacro:macro>
-<!-- Hokuyo Laser - CENTER -->
-    <!-- <xacro:macro name="laser_center">
-        <gazebo reference="hokuyo_link_center">
-            <sensor type="ray" name="head_hokuyo_sensor">
-            <pose>0 0 0 0 0 0</pose>
-            <visualize>true</visualize>
-            <update_rate>20</update_rate>
-            <ray>
-                <scan>
-                    <horizontal>
-                        <samples>360</samples>
-                        <resolution>1</resolution>
-                        <min_angle>-3.14</min_angle>
-                        <max_angle>3.14</max_angle>
-                    </horizontal>
-                </scan>
-                <range>
-                    <min>0.10</min>
-                    <max>10.0</max>
-                    <resolution>0.05</resolution>
-                </range>
-                <noise>
-                    <type>gaussian</type>
-                    <mean>0.0</mean>
-                    <stddev>0.01</stddev>
-                </noise>
-            </ray>
-            <plugin name="gazebo_ros_head_hokuyo_controller" filename="libgazebo_ros_laser.so">
-                <topicName>/scan_center</topicName>
-                <frameName>hokuyo_link_center</frameName>
-            </plugin>
-            </sensor>
-        </gazebo>
-        <link name="hokuyo_link_center">
-            <collision>
-                <origin xyz="0 0 0" rpy="0 0 0"/>
-                <geometry>
-                    <box size="0.1 0.1 0.1"/>
-                </geometry>
-            </collision>
-            <visual>
-                <origin xyz="0 0 0" rpy="0 0 0"/>
-                <geometry>
-                </geometry>
-            </visual>
-            <inertial>
-                <mass value="1e-5" />
-                <origin xyz="0 0 0" rpy="0 0 0"/>
-                <inertia ixx="1e-6" ixy="0" ixz="0" iyy="1e-6" iyz="0" izz="1e-6" />
-            </inertial>
-        </link>
-        <joint name="laser_joint_center" type="fixed">
-            <origin xyz="0.0 0 -0.28" rpy="0 0 0"/>
-            <parent link="chasis"/>
-            <child link="hokuyo_link_center"/>
-        </joint>
-    </xacro:macro> -->
-    <!-- Hokuyo Laser - LEFT -->
-    <xacro:macro name="laser_left">
-        <gazebo reference="hokuyo_link_left">
-            <sensor type="ray" name="head_hokuyo_sensor_left">
-            <pose>0 0 0 0 0 0</pose>
-            <visualize>true</visualize>
-            <update_rate>20</update_rate>
-            <ray>
-                <scan>
-                    <horizontal>
-                        <samples>50</samples>
-                        <resolution>1</resolution>
-                        <min_angle>-1.5</min_angle>
-                        <max_angle>1.5</max_angle>
-                    </horizontal>
-                </scan>
-                <range>
-                    <min>0.10</min>
-                    <max>10.0</max>
-                    <resolution>0.05</resolution>
-                </range>
-                <noise>
-                    <type>gaussian</type>
-                    <mean>0.0</mean>
-                    <stddev>0.01</stddev>
-                </noise>
-            </ray>
-            <plugin name="gazebo_ros_head_hokuyo_controller" filename="libgazebo_ros_laser.so">
-                <topicName>/scan_left</topicName>
-                <frameName>hokuyo_link_left</frameName>
-            </plugin>
-            </sensor>
-        </gazebo>
-        <link name="hokuyo_link_left">
-            <collision>
-                <origin xyz="0 0 0" rpy="0 0 0"/>
-                <geometry>
-                    <box size="0.1 0.1 0.1"/>
-                </geometry>
-            </collision>
-            <visual>
-                <origin xyz="0 0 0" rpy="0 0 0"/>
-                <geometry>
-                    <mesh filename="package://sweep_bot/meshes/hokuyo.dae"/>
-                </geometry>
-            </visual>
-            <inertial>
-                <mass value="1e-5" />
-                <origin xyz="0 0 0" rpy="0 0 0"/>
-                <inertia ixx="1e-6" ixy="0" ixz="0" iyy="1e-6" iyz="0" izz="1e-6" />
-            </inertial>
-        </link>
-        <joint name="laser_joint_left" type="fixed">
-            <origin xyz="0.0 0.25 -0.20" rpy="0 0.01 ${3.14/2}"/>
-            <parent link="chasis"/>
-            <child link="hokuyo_link_left"/>
-        </joint>
-    </xacro:macro>
-    <!-- Hokuyo Laser - RIGHT -->
-    <xacro:macro name="laser_right">
-        <gazebo reference="hokuyo_link_right">
-            <sensor type="ray" name="head_hokuyo_sensor_right">
-            <pose>0 0 0 0 0 0</pose>
-            <visualize>true</visualize>
-            <update_rate>20</update_rate>
-            <ray>
-                <scan>
-                    <horizontal>
-                        <samples>50</samples>
-                        <resolution>1</resolution>
-                        <min_angle>-1.5</min_angle>
-                        <max_angle>1.5</max_angle>
-                    </horizontal>
-                </scan>
-                <range>
-                    <min>0.10</min>
-                    <max>10.0</max>
-                    <resolution>0.05</resolution>
-                </range>
-                <noise>
-                    <type>gaussian</type>
-                    <mean>0.0</mean>
-                    <stddev>0.01</stddev>
-                </noise>
-            </ray>
-            <plugin name="gazebo_ros_head_hokuyo_controller" filename="libgazebo_ros_laser.so">
-                <topicName>/scan_right</topicName>
-                <frameName>hokuyo_link_right</frameName>
-            </plugin>
-            </sensor>
-        </gazebo>
-        <link name="hokuyo_link_right">
-            <collision>
-                <origin xyz="0 0 0" rpy="0 0 0"/>
-                <geometry>
-                    <box size="0.1 0.1 0.1"/>
-                </geometry>
-            </collision>
-            <visual>
-                <origin xyz="0 0 0" rpy="0 0 0"/>
-                <geometry>
-                    <mesh filename="package://sweep_bot/meshes/hokuyo.dae"/>
-                </geometry>
-            </visual>
-            <inertial>
-                <mass value="1e-5" />
-                <origin xyz="0 0 0" rpy="0 0 0"/>
-                <inertia ixx="1e-6" ixy="0" ixz="0" iyy="1e-6" iyz="0" izz="1e-6" />
-            </inertial>
-        </link>
-        <joint name="laser_joint_right" type="fixed">
-            <origin xyz="0.0 -0.25 -0.20" rpy="0 0.01 -${3.14/2}"/>
-            <parent link="chasis"/>
-            <child link="hokuyo_link_right"/>
-        </joint>
-    </xacro:macro>
-    <!-- Hokuyo Laser - REAR -->
-    <!-- <xacro:macro name="laser_rear">
-        <gazebo reference="hokuyo_link_rear">
-            <sensor type="ray" name="head_hokuyo_sensor_rear">
-            <pose>0 0 0 0 0 0</pose>
-            <visualize>true</visualize>
-            <update_rate>20</update_rate>
-            <ray>
-                <scan>
-                    <horizontal>
-                        <samples>720</samples>
-                        <resolution>1</resolution>
-                        <min_angle>-1.5</min_angle>
-                        <max_angle>1.5</max_angle>
-                    </horizontal>
-                </scan>
-                <range>
-                    <min>0.10</min>
-                    <max>10.0</max>
-                    <resolution>0.05</resolution>
-                </range>
-                <noise>
-                    <type>gaussian</type>
-                    <mean>0.0</mean>
-                    <stddev>0.01</stddev>
-                </noise>
-            </ray>
-            <plugin name="gazebo_ros_head_hokuyo_controller" filename="libgazebo_ros_laser.so">
-                <topicName>/scan_rear</topicName>
-                <frameName>hokuyo_link_rear</frameName>
-            </plugin>
-            </sensor>
-        </gazebo>
-        <link name="hokuyo_link_rear">
-            <collision>
-                <origin xyz="0 0 0" rpy="0 0 0"/>
-                <geometry>
-                    <box size="0.1 0.1 0.1"/>
-                </geometry>
-            </collision>
-            <visual>
-                <origin xyz="0 0 0" rpy="0 0 0"/>
-                <geometry>
-                    <mesh filename="package://sweep_bot/meshes/hokuyo.dae"/>
-                </geometry>
-            </visual>
-            <inertial>
-                <mass value="1e-5" />
-                <origin xyz="0 0 0" rpy="0 0 0"/>
-                <inertia ixx="1e-6" ixy="0" ixz="0" iyy="1e-6" iyz="0" izz="1e-6" />
-            </inertial>
-        </link>
-        <joint name="laser_joint_rear" type="fixed">
-            <origin xyz="-0.53 0 -0.20" rpy="0 0.01 ${3.14}"/>
-            <parent link="chasis"/>
-            <child link="hokuyo_link_rear"/>
-        </joint>
-    </xacro:macro> -->
-    <!-- ************************************************************** -->
     <!-- Hokuyo Laser - LEFT -->
     <xacro:macro name="laser_left_alt">
@@ -401,7 +54,5 @@
         </link>
         <joint name="laser_joint_left" type="fixed">
-            <!-- <origin xyz="0.5 0.25 -0.2" rpy="0.0 0.01 ${3.14/2}"/> -->
-            <!-- <origin xyz="0.53 0.25 0.2" rpy="0.0 0.01 ${3.14/2}"/> -->
-            <origin xyz="0.56 0.28 0.2" rpy="0.0 0.0 ${3.14/2}"/>
+            <origin xyz="0.56 0.28 -0.2" rpy="0.0 0.01 ${3.14/2}"/>
             <parent link="chasis"/>
             <child link="hokuyo_link_left"/>
@@ -461,7 +112,5 @@
         </link>
         <joint name="laser_joint_right" type="fixed">
-            <!-- <origin xyz="-0.5 -0.25 -0.2" rpy="0 0.01 -${3.14/2}"/> -->
-            <!-- <origin xyz="-0.53 -0.25 0.2" rpy="0.0 0.01 -${3.14/2}"/> -->
-            <origin xyz="-0.56 -0.28 0.2" rpy="0.0 0.0 -${3.14/2}"/>
+            <origin xyz="-0.56 -0.28 -0.2" rpy="0 0.01 -${3.14/2}"/>
             <parent link="chasis"/>
             <child link="hokuyo_link_right"/>
